Commit message: viz scanner model in rviz

File: src/pf_description/urdf/r2000.urdf.xacro (robot description, xacro)
@@ -6,5 +6,5 @@
                 <origin xyz="0 0 0" rpy="0 0 0" />
                 <geometry>
-                    <mesh filename="$(find pf_description)/meshes/R2000.dae" />
+                    <mesh filename="package://pf_description/meshes/R2000.stl" scale="0.001 0.001 0.001" />
                 </geometry>
             </visual>

File: src/pf_description/urdf/r2300.urdf.xacro (robot description, xacro)
@@ -6,5 +6,5 @@
                 <origin xyz="0 0 0" rpy="0 0 0" />
                 <geometry>
-                    <mesh filename="$(find pf_description)/meshes/R2300.dae" />
+                    <mesh filename="package://pf_description/meshes/R2300.stl" scale="0.001 0.001 0.001" />
                 </geometry>
             </visual>
